File: oled_ui.brd (EAGLE design)
At the start: 84.5 x 19.4 mm, 25 parts, among them IC1 74HC14D

Commit message: stuff
Parts:
- moved JP1 1.27 mm to (3.17, 15.2)
- moved JP2 1.27 mm to (81.3, 15.2)
Routing:
- net GND: track 0.00 -> 7.88 mm, vias 0 -> 2
- net BUTTONS_OUT2: track 18.3 -> 19.6 mm
- net RST: track 54.4 -> 53.9 mm
- net BUTTONS_OUT1: track 11.2 -> 11.8 mm
- net SCL: track 46.8 -> 46.2 mm
- net 3V3: track 72.9 -> 72.4 mm
Other:
- board size 84.5 x 19.4 mm -> 84.5 x 19.2 mm
Changed lines of the file:
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@@
 <plain>
 <wire x1="0" y1="19.05" x2="0" y2="4.445" width="0.4064" layer="20"/>
-<wire x1="0" y1="4.445" x2="2.54" y2="1.905" width="0.4064" layer="20" curve="90"/>
-<wire x1="2.54" y1="1.905" x2="33.02" y2="1.905" width="0.4064" layer="20"/>
-<wire x1="49.53" y1="1.905" x2="82.55" y2="1.905" width="0.4064" layer="20"/>
+<wire x1="0" y1="4.445" x2="1.9812" y2="2.1336" width="0.4064" layer="20" curve="90"/>
+<wire x1="1.9812" y1="2.1336" x2="33.7312" y2="2.1336" width="0.4064" layer="20"/>
+<wire x1="49.0728" y1="2.0828" x2="83.3628" y2="2.0828" width="0.4064" layer="20"/>
 <wire x1="0" y1="19.05" x2="2.6416" y2="21.2852" width="0.4064" layer="20" curve="-90"/>
 <wire x1="2.6416" y1="21.2852" x2="82.6516" y2="21.2852" width="0.4064" layer="20"/>
 <wire x1="82.6516" y1="21.2852" x2="84.455" y2="19.05" width="0.4064" layer="20" curve="-90"/>
 <wire x1="84.455" y1="19.05" x2="84.455" y2="3.81" width="0.4064" layer="20"/>
-<wire x1="84.455" y1="3.81" x2="82.55" y2="1.905" width="0.4064" layer="20" curve="-90"/>
+<wire x1="84.455" y1="3.81" x2="83.3628" y2="2.0828" width="0.4064" layer="20" curve="-90"/>
 <wire x1="34.29" y1="4.826" x2="48.26" y2="4.826" width="0.4064" layer="20"/>
 <wire x1="34.29" y1="4.826" x2="34.29" y2="3.175" width="0.4064" layer="20"/>
-<wire x1="34.29" y1="3.175" x2="33.02" y2="1.905" width="0.4064" layer="20" curve="-90"/>
+<wire x1="34.29" y1="3.175" x2="33.7312" y2="2.1336" width="0.4064" layer="20" curve="-90"/>
 <wire x1="48.26" y1="4.826" x2="48.26" y2="3.175" width="0.4064" layer="20"/>
-<wire x1="48.26" y1="3.175" x2="49.53" y2="1.905" width="0.4064" layer="20" curve="90"/>
-<text x="80.7974" y="2.7686" size="1.016" layer="25" font="vector">GND
+<wire x1="48.26" y1="3.175" x2="49.0728" y2="2.0828" width="0.4064" layer="20" curve="90"/>
+<text x="80.7974" y="4.0386" size="1.016" layer="25" font="vector">GND
 IN1
 IN2
 3V3</text>
-<text x="1.4224" y="2.7686" size="1.016" layer="25" font="vector">GND
+<text x="1.4224" y="4.0386" size="1.016" layer="25" font="vector">GND
 SDA
 SCL
 RST</text>
-<text x="3.9624" y="2.7686" size="1.016" layer="26" font="vector" rot="MR0">GND
+<text x="3.9624" y="4.0386" size="1.016" layer="26" font="vector" rot="MR0">GND
 SDA
 SCL
 RST</text>
-<text x="83.3374" y="2.7686" size="1.016" layer="26" font="vector" rot="MR0">GND
+<text x="83.3374" y="4.0386" size="1.016" layer="26" font="vector" rot="MR0">GND
 IN1
 IN2
@@
 <attribute name="NAME" x="67.1449" y="10.6553" size="1.27" layer="25" ratio="10" rot="R180"/>
 </element>
-<element name="JP1" library="pinhead" package="1X04" value="" x="3.175" y="13.97" smashed="yes" rot="R90">
-<attribute name="NAME" x="4.5212" y="20.5867" size="1.27" layer="25" ratio="10" rot="R180"/>
-<attribute name="VALUE" x="6.35" y="8.89" size="1.27" layer="27" rot="R90"/>
-</element>
-<element name="JP2" library="pinhead" package="1X04" value="" x="81.28" y="13.97" smashed="yes" rot="R90">
-<attribute name="NAME" x="82.7151" y="20.6121" size="1.27" layer="25" ratio="10" rot="R180"/>
-<attribute name="VALUE" x="84.455" y="8.89" size="1.27" layer="27" rot="R90"/>
+<element name="JP1" library="pinhead" package="1X04" value="" x="3.175" y="15.24" smashed="yes" rot="R90">
+<attribute name="NAME" x="4.8133" y="6.4262" size="1.27" layer="25" ratio="10" rot="R270"/>
+<attribute name="VALUE" x="6.35" y="10.16" size="1.27" layer="27" rot="R90"/>
+</element>
+<element name="JP2" library="pinhead" package="1X04" value="" x="81.28" y="15.24" smashed="yes" rot="R90">
+<attribute name="NAME" x="78.4479" y="11.5951" size="1.27" layer="25" ratio="10" rot="R270"/>
+<attribute name="VALUE" x="84.455" y="10.16" size="1.27" layer="27" rot="R90"/>
 </element>
 <element name="C7" library="rcl" package="C0805" value="" x="39.1668" y="16.5227" smashed="yes" rot="R270">
@@
 <contactref element="JP2" pad="4"/>
 <contactref element="C7" pad="1"/>
+<wire x1="75.565" y1="8.3566" x2="77.3557" y2="8.3566" width="0.4064" layer="1"/>
+<wire x1="77.3684" y1="8.3566" x2="77.3557" y2="8.3566" width="0.4064" layer="1"/>
+<via x="77.3557" y="8.3566" extent="1-16" drill="0.7"/>
+<wire x1="77.3557" y1="8.3566" x2="75.4126" y2="8.3566" width="0.4064" layer="16"/>
+<wire x1="75.4126" y1="8.3566" x2="73.0123" y2="5.9055" width="0.4064" layer="16"/>
+<via x="73.0123" y="5.9055" extent="1-16" drill="0.6"/>
+<wire x1="73.0123" y1="5.9055" x2="72.5805" y2="5.9055" width="0.4064" layer="1"/>
+<wire x1="72.5805" y1="5.9055" x2="72.39" y2="5.715" width="0.4064" layer="1"/>
 </signal>
 <signal name="SDA">
@@
 <wire x1="11.0617" y1="17.145" x2="10.8077" y2="16.891" width="0.4064" layer="16"/>
 <wire x1="10.8077" y1="16.891" x2="10.8077" y2="11.4427" width="0.4064" layer="16"/>
-<wire x1="10.8077" y1="11.4427" x2="9.525" y2="10.16" width="0.4064" layer="16"/>
-<wire x1="9.525" y1="10.16" x2="3.175" y2="10.16" width="0.4064" layer="16"/>
 <wire x1="38.7988" y1="9.7298" x2="38.7861" y2="11.4805" width="0.4064" layer="1"/>
 <wire x1="38.7861" y1="11.4805" x2="38.1" y2="12.065" width="0.4064" layer="1"/>
+<wire x1="3.175" y1="11.43" x2="3.81" y2="10.795" width="0.4064" layer="16"/>
+<wire x1="3.81" y1="10.795" x2="10.16" y2="10.795" width="0.4064" layer="16"/>
+<wire x1="10.16" y1="10.795" x2="10.8077" y2="11.4427" width="0.4064" layer="16"/>
 </signal>
 <signal name="SCL">
@@
 <wire x1="39.4843" y1="15.7607" x2="37.465" y2="17.78" width="0.4064" layer="16"/>
 <contactref element="JP1" pad="2"/>
-<wire x1="9.525" y1="13.97" x2="4.445" y2="13.97" width="0.4064" layer="16"/>
-<wire x1="4.445" y1="13.97" x2="3.175" y2="12.7" width="0.4064" layer="16"/>
+<wire x1="9.525" y1="13.97" x2="3.175" y2="13.97" width="0.4064" layer="16"/>
 </signal>
 <signal name="3V3">
@@
 <wire x1="66.675" y1="6.985" x2="66.675" y2="10.16" width="0.4064" layer="1"/>
 <contactref element="JP2" pad="1"/>
-<wire x1="81.28" y1="10.16" x2="75.565" y2="10.16" width="0.6096" layer="1"/>
-<wire x1="75.565" y1="10.16" x2="74.295" y2="11.43" width="0.6096" layer="1"/>
-<wire x1="74.295" y1="11.43" x2="66.675" y2="11.43" width="0.6096" layer="1"/>
+<wire x1="81.28" y1="11.43" x2="66.675" y2="11.43" width="0.6096" layer="1"/>
 <wire x1="67.945" y1="13.97" x2="67.31" y2="13.97" width="0.6096" layer="1"/>
 <wire x1="67.31" y1="13.97" x2="66.675" y2="13.335" width="0.6096" layer="1"/>
@@
 <wire x1="42.2783" y1="15.5727" x2="41.656" y2="15.56" width="0.4064" layer="1"/>
 <contactref element="JP1" pad="3"/>
-<wire x1="3.175" y1="15.24" x2="3.81" y2="15.24" width="0.4064" layer="16"/>
-<wire x1="3.81" y1="15.24" x2="5.715" y2="17.145" width="0.4064" layer="16"/>
-<wire x1="5.715" y1="17.145" x2="8.89" y2="17.145" width="0.4064" layer="16"/>
+<wire x1="3.81" y1="17.145" x2="8.89" y2="17.145" width="0.4064" layer="16"/>
 <wire x1="8.89" y1="17.145" x2="10.16" y2="18.415" width="0.4064" layer="16"/>
 <wire x1="10.16" y1="18.415" x2="37.8997" y2="18.415" width="0.4064" layer="16"/>
@@
 <via x="42.2988" y="12.065" extent="1-16" drill="0.6"/>
 <wire x1="42.2988" y1="12.065" x2="42.2988" y2="14.0159" width="0.4064" layer="1"/>
+<wire x1="3.81" y1="17.145" x2="3.175" y2="16.51" width="0.4064" layer="16"/>
 </signal>
 <signal name="N$11">
@@
 <contactref element="JP2" pad="3"/>
 <wire x1="76.2" y1="18.98" x2="76.9728" y2="18.98" width="0.4064" layer="1"/>
-<wire x1="81.28" y1="15.24" x2="76.835" y2="15.24" width="0.4064" layer="16"/>
-<wire x1="76.835" y1="15.24" x2="76.2" y2="15.875" width="0.4064" layer="16"/>
 <wire x1="76.2" y1="15.875" x2="76.2" y2="19.685" width="0.4064" layer="16"/>
 <via x="76.2" y="19.685" extent="1-16" drill="0.6"/>
 <wire x1="76.2" y1="19.685" x2="76.2" y2="18.98" width="0.4064" layer="1"/>
+<wire x1="76.2" y1="15.875" x2="76.835" y2="15.24" width="0.4064" layer="16"/>
+<wire x1="76.835" y1="15.24" x2="79.375" y2="15.24" width="0.4064" layer="16"/>
+<wire x1="79.375" y1="15.24" x2="80.645" y2="16.51" width="0.4064" layer="16"/>
+<wire x1="80.645" y1="16.51" x2="81.28" y2="16.51" width="0.4064" layer="16"/>
 </signal>
 <signal name="BUTTONS_OUT2">
@@
 <wire x1="80.01" y1="3.81" x2="80.01" y2="6.985" width="0.4064" layer="16"/>
 <wire x1="80.01" y1="6.985" x2="78.74" y2="8.255" width="0.4064" layer="16"/>
-<wire x1="78.74" y1="8.255" x2="78.74" y2="12.065" width="0.4064" layer="16"/>
-<wire x1="78.74" y1="12.065" x2="79.375" y2="12.7" width="0.4064" layer="16"/>
-<wire x1="79.375" y1="12.7" x2="81.28" y2="12.7" width="0.4064" layer="16"/>
+<wire x1="78.74" y1="8.255" x2="78.74" y2="13.335" width="0.4064" layer="16"/>
+<wire x1="81.28" y1="13.97" x2="79.375" y2="13.97" width="0.4064" layer="16"/>
+<wire x1="79.375" y1="13.97" x2="78.74" y2="13.335" width="0.4064" layer="16"/>
 </signal>
 <signal name="N$26">

Commit message: big flip
Parts:
- moved U$1 26.7 mm to (27.9, -5.08), flipped to the top
- moved C6 22.4 mm to (30.1, 17.2), flipped to the bottom, turned to 270 degrees
- moved C3 22.2 mm to (52.2, 17.1), flipped to the bottom
- moved C5 16.7 mm to (33.2, 17.1), flipped to the bottom, turned to 270 degrees
- moved C4 16.5 mm to (49.4, 17.1), flipped to the bottom
- moved C2 11.9 mm to (35.5, 17.1), flipped to the bottom
- moved R1 10.2 mm to (46.1, 17.1), flipped to the bottom
- moved C1 6.38 mm to (38.0, 17.1), flipped to the bottom
- moved C7 4.49 mm to (43.6, 17.2), flipped to the bottom
- moved RN1 1.42 mm to (67.3, 4.45), flipped to the bottom, turned to 270 degrees
- moved RN2 1.42 mm to (67.3, 18.4), flipped to the bottom, turned to 270 degrees
- moved R2 0.90 mm to (41.0, 17.1), flipped to the bottom
- moved RN6 0.64 mm to (77.7, 18.4), flipped to the bottom, turned to 270 degrees
- moved RN3 0.63 mm to (74.9, 4.45), flipped to the bottom, turned to 90 degrees
- moved RN4 0.63 mm to (74.9, 18.4), flipped to the bottom, turned to 90 degrees
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- renumbered S1 to E, S2 to F, S3 to B, S4 to A, S5 to D, S6 to C
Connections:
- net N$11: now also C.1
- net N$12: now also D.1
- net N$5: now also B.1
- net N$9: now also A.1
- net RST: now also JP1.1; no longer JP1.3
- net SDA: now also JP1.3; no longer JP1.1
Routing:
- net GND: track 7.88 -> 32.4 mm, vias 2 -> 3
- net N$14: track 15.5 -> 36.1 mm, vias 1 -> 2
- net N$11: track 70.1 -> 88.5 mm, vias 1 -> 2
- net N$5: track 71.1 -> 84.3 mm, vias 1 -> 2
- net 3V3: track 72.4 -> 84.1 mm
- net SCL: track 46.2 -> 56.9 mm, vias 1 -> 0
- net N$19: track 12.6 -> 2.73 mm, vias 2 -> 0
- net N$9: track 81.6 -> 91.0 mm, vias 1 -> 2
- net N$17: track 2.70 -> 10.3 mm
- net N$20: track 2.09 -> 8.99 mm
- net BUTTONS_OUT2: track 19.6 -> 13.4 mm
- net BUTTONS_OUT1: track 11.8 -> 6.29 mm, vias 1 -> 0
- net N$15: track 8.16 -> 3.53 mm, vias 2 -> 0
- net N$2: track 6.54 -> 11.1 mm
- net N$3: track 6.04 -> 10.4 mm
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- added copper zone on layer 16, net GND
