File: oled_ui.sch (EAGLE design)
At the start: 30 parts

Commit message: updates
Parts:
- removed J1: (no value), tag-connect:TC2030-MCP-NL
- removed R2R1, R2R2, R2R3, R2R45, R2R56, R2R6, RR1, RR2, RR3, RR4, RR5, RR6: (no value), rcl:R-EU_R0805
- removed U$2: PIC12F1822SO08, jasons_stuff:PIC12F1822SO08
- added IC1: 74HC14D, 74xx-eu:74HC14D
- added JP2: (no value), pinhead:PINHD-1X4
- added R2: (no value), rcl:R-EU_R0805
- added RN1, RN2, RN3, RN4, RN5, RN6: (no value), resistor-dil:4R-NCAY16
- C2, C5, C6: device resistor:CPOL-EUSMCA -> rcl:C-EUC0805
- JP1: device pinhead:PINHD-2X3 -> pinhead:PINHD-1X4
Connections:
- removed net IRQ: JP1.2, U$2.RA5
- removed net OLED_RST: JP1.5, U$1.RES#
- removed net VDD: C1.+, C7.1, J1.VDD, JP1.4, S1.P, S1.P1, S2.P, S2.P1, S3.P, S3.P1, S4.P, S4.P1, S5.P, S5.P1, S6.P, S6.P1, U$1.BS1, U$1.VDD, U$2.VDD
- new net 3V3: C1.+, IC1P.VCC, JP2.1, R2.2, RN1A.2, RN1B.1, RN1B.2, RN1C.2, RN1D.2, RN2A.2, RN2B.1, RN2B.2, RN2C.2, RN2D.2, U$1.BS1, U$1.VDD
- new net BUTTONS_OUT1: JP2.3, RN4A.2, RN6D.2
- new net BUTTONS_OUT2: JP2.2, RN3D.2, RN5A.2
- new net N$22: RN4C.2, RN4D.2, RN6A.1, RN6A.2, RN6B.1, RN6B.2, RN6C.1
- new net N$23: RN3C.2, RN5A.1, RN5B.2
- new net N$26: RN3A.2, RN3B.2, RN5B.1, RN5C.1, RN5C.2, RN5D.1, RN5D.2
- new net RST: C7.2, JP1.1, R2.1, U$1.RES#
- net GND: now also C2.2, C7.1, IC1P.GND, JP1.4, JP2.4, RN3B.1, RN4C.1, S1.P, S1.P1, S2.P, S2.P1, S3.P, S3.P1, S4.P, S4.P1, S5.P, S5.P1, S6.P, S6.P1; no longer C2.-, C7.2, J1.VSS(GND), JP1.6, R2R3.1, R2R6.1, U$2.VSS
- net N$1: now also C6.2; no longer C6.-
- net N$11: now also IC1D.I, RN1D.1, S6.S1; no longer RR1.1, S1.S, S1.S1
- net N$12: now also IC1C.I, RN2D.1, S5.S1; no longer R2R45.2, RR4.2, U$2.RA4
- net N$13: now also IC1B.I, RN2C.1, S1.S, S1.S1; no longer RR2.1, S2.S, S2.S1
- net N$14: now also IC1A.I, RN2A.1, S2.S, S2.S1; no longer RR6.1, S6.S, S6.S1
- net N$15: now also IC1A.O, RN4A.1; no longer RR5.1, S5.S, S5.S1
- net N$16: now also IC1B.O, RN4B.1; no longer RR4.1, S4.S, S4.S1
- net N$17: now also IC1C.O, RN4D.1; no longer RR3.1, S3.S, S3.S1
- net N$18: now also IC1E.O, RN3C.1; no longer J1.ICSP_DAT/PGD, R2R1.1, RR1.2, U$2.RA0/PGD
- net N$19: now also IC1D.O, RN3D.1; no longer R2R1.2, R2R2.2, RR2.2
- net N$2: now also C6.1; no longer C6.+
- net N$20: now also IC1F.O, RN3A.1; no longer R2R2.1, R2R3.2, RR3.2
- net N$21: now also RN4B.2, RN6C.2, RN6D.1; no longer J1.VPP/MCLR, U$2.MCLR#/VPP/RA3
- net N$3: now also C5.1; no longer C5.+
- net N$4: now also C5.2; no longer C5.-
- net N$5: now also IC1F.I, RN1A.1, S3.S1; no longer R2R56.1, R2R6.2, RR6.2
- net N$7: now also C2.1; no longer C2.+
- net N$9: now also IC1E.I, RN1C.1, S4.S1; no longer R2R45.1, R2R56.2, RR5.2
- net SCL: now also JP1.2; no longer J1.ICSP_CLK/PGC, JP1.1, U$2.RA1/PGC
- net SDA: no longer U$2.RA2
Other:
- moved on the sheet: C7, S1, S2, S3, S4, S5, S6

Commit message: OOPS!
Connections:
- net RST: now also JP1.3; no longer JP1.1
- net SDA: now also JP1.1; no longer JP1.3
Changed lines of the file:
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@@
 </segment>
 <segment>
-<label x="109.22" y="0" size="1.778" layer="95"/>
-<wire x1="121.92" y1="0" x2="111.76" y2="0" width="0.1524" layer="91"/>
-<pinref part="JP1" gate="A" pin="3"/>
-<junction x="121.92" y="0"/>
+<label x="106.68" y="5.08" size="1.778" layer="95"/>
+<pinref part="JP1" gate="A" pin="1"/>
+<wire x1="111.76" y1="5.08" x2="121.92" y2="5.08" width="0.1524" layer="91"/>
+<junction x="121.92" y="5.08"/>
 </segment>
 </net>
@@
 <segment>
 <label x="106.68" y="2.54" size="1.778" layer="95"/>
-<wire x1="121.92" y1="2.54" x2="111.76" y2="2.54" width="0.1524" layer="91"/>
 <pinref part="JP1" gate="A" pin="2"/>
+<wire x1="111.76" y1="2.54" x2="121.92" y2="2.54" width="0.1524" layer="91"/>
 <junction x="121.92" y="2.54"/>
 </segment>
@@
 </segment>
 <segment>
-<pinref part="JP1" gate="A" pin="1"/>
-<wire x1="121.92" y1="5.08" x2="99.06" y2="5.08" width="0.1524" layer="91"/>
-<label x="99.06" y="5.08" size="1.778" layer="95"/>
-<junction x="121.92" y="5.08"/>
+<label x="106.68" y="0" size="1.778" layer="95"/>
+<wire x1="121.92" y1="0" x2="99.06" y2="0" width="0.1524" layer="91"/>
+<pinref part="JP1" gate="A" pin="3"/>
+<junction x="121.92" y="0"/>
 </segment>
 </net>

Commit message: big flip
Parts:
- renumbered S1 to E, S2 to F, S3 to B, S4 to A, S5 to D, S6 to C
Connections:
- net N$11: now also C.S
- net N$12: now also D.S
- net N$5: now also B.S
- net N$9: now also A.S
- net RST: now also JP1.1; no longer JP1.3
- net SDA: now also JP1.3; no longer JP1.1

Commit message: updates in progress
Parts:
- removed RN1, RN2, RN3, RN4, RN5, RN6: (no value), resistor-dil:4R-NCAY16
- added D1: 0805DIODE, jasons_stuff:0805DIODE
- added R10, R3, R4, R5, R6, R7, R8, R9, RA1, RA2, RA3, RA4, RA5, RA6, RA7, RB1, RB2, RB3, RB4, RB5, RB6: (no value), rcl:R-EU_R0805
- added U1: (no value), microbuilder:VREG_SOT23
- C1, C3: device resistor:CPOL-EUSMCA -> rcl:C-EUC0805
- C4: device resistor:CPOL-EUSMCB -> rcl:C-EUC0805
Connections:
- removed net N$19: IC1D.O, RN3D.1
- removed net N$26: RN3A.2, RN3B.2, RN5B.1, RN5C.1, RN5C.2, RN5D.1, RN5D.2
- new net 5V: C2.1, IC1P.VCC, JP2.1, R3.2, R4.2, R5.2, R6.2, R7.2, R8.2, U1.VIN
- new net N$24: IC1A.O, RA1.2
- net 3V3: now also C1.1, D1.P$2, R10.1, R9.1, U$1.VBAT, U1.VOUT; no longer C1.+, IC1P.VCC, JP2.1, RN1A.2, RN1B.1, RN1B.2, RN1C.2, RN1D.2, RN2A.2, RN2B.1, RN2B.2, RN2C.2, RN2D.2
- net BUTTONS_OUT1: now also RA1.1, RB1.1; no longer RN4A.2, RN6D.2
- net BUTTONS_OUT2: now also RA4.2, RA5.1, RB4.1; no longer RN3D.2, RN5A.2
- net GND: now also C1.2, C3.2, C4.2, RB3.2, RB6.2, U$1.CS#, U$1.D3, U$1.D4, U$1.D5, U$1.D6, U$1.D7, U$1.E/RD#, U$1.NC, U$1.R/W#, U1.GND; no longer C1.-, C3.-, C4.-, RN3B.1, RN4C.1
- net N$11: now also R6.1; no longer RN1D.1
- net N$12: now also R5.1; no longer RN2D.1
- net N$13: now also R4.1; no longer RN2C.1
- net N$14: now also R3.1; no longer RN2A.1
- net N$15: now also IC1E.O, RA6.2; no longer IC1A.O, RN4A.1
- net N$16: now also IC1F.O, RA7.2; no longer IC1B.O, RN4B.1
- net N$17: now also RA7.1, RB5.2, RB6.1; no longer IC1C.O, RN4D.1
- net N$18: now also RA6.1, RB4.2, RB5.1; no longer IC1E.O, RN3C.1
- net N$20: now also IC1C.O, RA3.2; no longer IC1F.O, RN3A.1
- net N$21: now also RA3.1, RA4.1, RB2.2, RB3.1; no longer RN4B.2, RN6C.2, RN6D.1
- net N$22: now also IC1B.O, RA2.2; no longer RN4C.2, RN4D.2, RN6A.1, RN6A.2, RN6B.1, RN6B.2, RN6C.1
- net N$23: now also RA2.1, RB1.2, RB2.1; no longer RN3C.2, RN5A.1, RN5B.2
- net N$5: now also R8.1; no longer RN1A.1
- net N$6: now also C3.1; no longer C3.+
- net N$7: now also IC1D.O, RA5.2; no longer C2.1, U$1.VBAT
- net N$8: now also C4.1; no longer C4.+
- net N$9: now also R7.1; no longer RN1C.1
- net RST: now also D1.P$1
- net SCL: now also R9.2
- net SDA: now also R10.2
Other:
- moved on the sheet: C2, C7

Commit message: Revert "updates in progress"
This reverts commit 001d56b77ca17e324d01e8b0934cb9d53080aba6.
Parts:
- removed D1: 0805DIODE, jasons_stuff:0805DIODE
- removed R10, R3, R4, R5, R6, R7, R8, R9, RA1, RA2, RA3, RA4, RA5, RA6, RA7, RB1, RB2, RB3, RB4, RB5, RB6: (no value), rcl:R-EU_R0805
- removed U1: (no value), microbuilder:VREG_SOT23
- added RN1, RN2, RN3, RN4, RN5, RN6: (no value), resistor-dil:4R-NCAY16
- C1, C3: device rcl:C-EUC0805 -> resistor:CPOL-EUSMCA
- C4: device rcl:C-EUC0805 -> resistor:CPOL-EUSMCB
Connections:
- removed net 5V: C2.1, IC1P.VCC, JP2.1, R3.2, R4.2, R5.2, R6.2, R7.2, R8.2, U1.VIN
- removed net N$24: IC1A.O, RA1.2
- new net N$19: IC1D.O, RN3D.1
- new net N$26: RN3A.2, RN3B.2, RN5B.1, RN5C.1, RN5C.2, RN5D.1, RN5D.2
- net 3V3: now also C1.+, IC1P.VCC, JP2.1, RN1A.2, RN1B.1, RN1B.2, RN1C.2, RN1D.2, RN2A.2, RN2B.1, RN2B.2, RN2C.2, RN2D.2; no longer C1.1, D1.P$2, R10.1, R9.1, U$1.VBAT, U1.VOUT
- net BUTTONS_OUT1: now also RN4A.2, RN6D.2; no longer RA1.1, RB1.1
- net BUTTONS_OUT2: now also RN3D.2, RN5A.2; no longer RA4.2, RA5.1, RB4.1
- net GND: now also C1.-, C3.-, C4.-, RN3B.1, RN4C.1; no longer C1.2, C3.2, C4.2, RB3.2, RB6.2, U$1.CS#, U$1.D3, U$1.D4, U$1.D5, U$1.D6, U$1.D7, U$1.E/RD#, U$1.NC, U$1.R/W#, U1.GND
- net N$11: now also RN1D.1; no longer R6.1
- net N$12: now also RN2D.1; no longer R5.1
- net N$13: now also RN2C.1; no longer R4.1
- net N$14: now also RN2A.1; no longer R3.1
- net N$15: now also IC1A.O, RN4A.1; no longer IC1E.O, RA6.2
- net N$16: now also IC1B.O, RN4B.1; no longer IC1F.O, RA7.2
- net N$17: now also IC1C.O, RN4D.1; no longer RA7.1, RB5.2, RB6.1
- net N$18: now also IC1E.O, RN3C.1; no longer RA6.1, RB4.2, RB5.1
- net N$20: now also IC1F.O, RN3A.1; no longer IC1C.O, RA3.2
- net N$21: now also RN4B.2, RN6C.2, RN6D.1; no longer RA3.1, RA4.1, RB2.2, RB3.1
- net N$22: now also RN4C.2, RN4D.2, RN6A.1, RN6A.2, RN6B.1, RN6B.2, RN6C.1; no longer IC1B.O, RA2.2
- net N$23: now also RN3C.2, RN5A.1, RN5B.2; no longer RA2.1, RB1.2, RB2.1
- net N$5: now also RN1A.1; no longer R8.1
- net N$6: now also C3.+; no longer C3.1
- net N$7: now also C2.1, U$1.VBAT; no longer IC1D.O, RA5.2
- net N$8: now also C4.+; no longer C4.1
- net N$9: now also RN1C.1; no longer R7.1
- net RST: no longer D1.P$1
- net SCL: no longer R9.2
- net SDA: no longer R10.2
Other:
- moved on the sheet: C2, C7

Commit message: work in progress
Parts:
- removed RN1, RN2, RN3, RN4, RN5, RN6: (no value), resistor-dil:4R-NCAY16
- added D1: 0805DIODE, jasons_stuff:0805DIODE
- added R10, R11, R12, R13, R14, R15, R16, R17, R18, R19, R20, R21, R22, R23, R3, R4, R5, R6, R7, R8, R9: (no value), rcl:R-EU_R0805
- added REG1: (no value), microbuilder:VREG_SOT23
- C1, C3: device resistor:CPOL-EUSMCA -> rcl:C-EUC0805
- C4: device resistor:CPOL-EUSMCB -> rcl:C-EUC0805
Connections:
- removed net N$19: IC1D.O, RN3D.1
- removed net N$26: RN3A.2, RN3B.2, RN5B.1, RN5C.1, RN5C.2, RN5D.1, RN5D.2
- new net 5V: C2.1, IC1P.VCC, JP2.1, R3.2, R4.2, R5.2, R6.2, R7.2, R8.2, REG1.VIN
- new net N$24: IC1A.O, R11.2
- net 3V3: now also C1.1, D1.P$2, R10.1, R9.1, REG1.VOUT, U$1.VBAT; no longer C1.+, IC1P.VCC, JP2.1, RN1A.2, RN1B.1, RN1B.2, RN1C.2, RN1D.2, RN2A.2, RN2B.1, RN2B.2, RN2C.2, RN2D.2
- net BUTTONS_OUT1: now also R11.1, R17.1; no longer RN4A.2, RN6D.2
- net BUTTONS_OUT2: now also R14.1, R20.2, R21.1; no longer RN3D.2, RN5A.2
- net GND: now also C1.2, C3.2, C4.2, R19.2, R23.2, REG1.GND, U$1.CS#, U$1.D3, U$1.D4, U$1.D5, U$1.D6, U$1.D7, U$1.E/RD#, U$1.NC, U$1.R/W#; no longer C1.-, C3.-, C4.-, RN3B.1, RN4C.1
- net N$11: now also R6.1; no longer RN1D.1
- net N$12: now also R5.1; no longer RN2D.1
- net N$13: now also R4.1; no longer RN2C.1
- net N$14: now also R3.1; no longer RN2A.1
- net N$15: now also IC1E.O, R15.2; no longer IC1A.O, RN4A.1
- net N$16: now also IC1F.O, R16.2; no longer IC1B.O, RN4B.1
- net N$17: now also R16.1, R22.2, R23.1; no longer IC1C.O, RN4D.1
- net N$18: now also R15.1, R21.2, R22.1; no longer IC1E.O, RN3C.1
- net N$20: now also IC1C.O, R13.2; no longer IC1F.O, RN3A.1
- net N$21: now also R13.1, R18.2, R19.1, R20.1; no longer RN4B.2, RN6C.2, RN6D.1
- net N$22: now also IC1B.O, R12.2; no longer RN4C.2, RN4D.2, RN6A.1, RN6A.2, RN6B.1, RN6B.2, RN6C.1
- net N$23: now also R12.1, R17.2, R18.1; no longer RN3C.2, RN5A.1, RN5B.2
- net N$5: now also R8.1; no longer RN1A.1
- net N$6: now also C3.1; no longer C3.+
- net N$7: now also IC1D.O, R14.2; no longer C2.1, U$1.VBAT
- net N$8: now also C4.1; no longer C4.+
- net N$9: now also R7.1; no longer RN1C.1
- net RST: now also D1.P$1
- net SCL: now also R9.2
- net SDA: now also R10.2
Other:
- moved on the sheet: C2, C7

Commit message: ready?
Parts:
- renumbered R11 to 8B, R12 to 7B, R13 to 6B, R14 to 4B, R15 to 3B, R16 to 2B, R17 to 4A, R18 to 3A, R19 to 5B, R20 to J1, R21 to 2A, R22 to 1A, R23 to 1B
Changed lines of the file:
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@@
 <part name="R7" library="rcl" deviceset="R-EU_" device="R0805"/>
 <part name="R8" library="rcl" deviceset="R-EU_" device="R0805"/>
-<part name="R11" library="rcl" deviceset="R-EU_" device="R0805"/>
-<part name="R12" library="rcl" deviceset="R-EU_" device="R0805"/>
-<part name="R13" library="rcl" deviceset="R-EU_" device="R0805"/>
-<part name="R14" library="rcl" deviceset="R-EU_" device="R0805"/>
-<part name="R15" library="rcl" deviceset="R-EU_" device="R0805"/>
-<part name="R16" library="rcl" deviceset="R-EU_" device="R0805"/>
-<part name="R23" library="rcl" deviceset="R-EU_" device="R0805"/>
-<part name="R22" library="rcl" deviceset="R-EU_" device="R0805"/>
-<part name="R21" library="rcl" deviceset="R-EU_" device="R0805"/>
-<part name="R20" library="rcl" deviceset="R-EU_" device="R0805"/>
-<part name="R19" library="rcl" deviceset="R-EU_" device="R0805"/>
-<part name="R18" library="rcl" deviceset="R-EU_" device="R0805"/>
-<part name="R17" library="rcl" deviceset="R-EU_" device="R0805"/>
+<part name="8B" library="rcl" deviceset="R-EU_" device="R0805"/>
+<part name="7B" library="rcl" deviceset="R-EU_" device="R0805"/>
+<part name="6B" library="rcl" deviceset="R-EU_" device="R0805"/>
+<part name="4B" library="rcl" deviceset="R-EU_" device="R0805"/>
+<part name="3B" library="rcl" deviceset="R-EU_" device="R0805"/>
+<part name="2B" library="rcl" deviceset="R-EU_" device="R0805"/>
+<part name="1B" library="rcl" deviceset="R-EU_" device="R0805"/>
+<part name="1A" library="rcl" deviceset="R-EU_" device="R0805"/>
+<part name="2A" library="rcl" deviceset="R-EU_" device="R0805"/>
+<part name="J1" library="rcl" deviceset="R-EU_" device="R0805"/>
+<part name="5B" library="rcl" deviceset="R-EU_" device="R0805"/>
+<part name="3A" library="rcl" deviceset="R-EU_" device="R0805"/>
+<part name="4A" library="rcl" deviceset="R-EU_" device="R0805"/>
 <part name="GND7" library="supply1" deviceset="GND" device=""/>
 <part name="R9" library="rcl" deviceset="R-EU_" device="R0805"/>
@@
 <instance part="R7" gate="G$1" x="101.6" y="-58.42" rot="R90"/>
 <instance part="R8" gate="G$1" x="104.14" y="-58.42" rot="R90"/>
-<instance part="R11" gate="G$1" x="134.62" y="-68.58" rot="R180"/>
-<instance part="R12" gate="G$1" x="134.62" y="-81.28" rot="R180"/>
-<instance part="R13" gate="G$1" x="134.62" y="-93.98" rot="R180"/>
-<instance part="R14" gate="G$1" x="134.62" y="-129.54" rot="R180"/>
-<instance part="R15" gate="G$1" x="134.62" y="-142.24" rot="R180"/>
-<instance part="R16" gate="G$1" x="134.62" y="-154.94" rot="R180"/>
-<instance part="R23" gate="G$1" x="142.24" y="-162.56" rot="R270"/>
-<instance part="R22" gate="G$1" x="142.24" y="-147.32" rot="R270"/>
-<instance part="R21" gate="G$1" x="142.24" y="-134.62" rot="R270"/>
-<instance part="R20" gate="G$1" x="152.4" y="-104.14" rot="R270"/>
-<instance part="R19" gate="G$1" x="142.24" y="-104.14" rot="R270"/>
-<instance part="R18" gate="G$1" x="142.24" y="-86.36" rot="R270"/>
-<instance part="R17" gate="G$1" x="142.24" y="-73.66" rot="R270"/>
+<instance part="8B" gate="G$1" x="134.62" y="-68.58" rot="R180"/>
+<instance part="7B" gate="G$1" x="134.62" y="-81.28" rot="R180"/>
+<instance part="6B" gate="G$1" x="134.62" y="-93.98" rot="R180"/>
+<instance part="4B" gate="G$1" x="134.62" y="-129.54" rot="R180"/>
+<instance part="3B" gate="G$1" x="134.62" y="-142.24" rot="R180"/>
+<instance part="2B" gate="G$1" x="134.62" y="-154.94" rot="R180"/>
+<instance part="1B" gate="G$1" x="142.24" y="-162.56" rot="R270"/>
+<instance part="1A" gate="G$1" x="142.24" y="-147.32" rot="R270"/>
+<instance part="2A" gate="G$1" x="142.24" y="-134.62" rot="R270"/>
+<instance part="J1" gate="G$1" x="152.4" y="-104.14" rot="R270"/>
+<instance part="5B" gate="G$1" x="142.24" y="-104.14" rot="R270"/>
+<instance part="3A" gate="G$1" x="142.24" y="-86.36" rot="R270"/>
+<instance part="4A" gate="G$1" x="142.24" y="-73.66" rot="R270"/>
 <instance part="GND7" gate="1" x="142.24" y="-111.76"/>
 <instance part="R9" gate="G$1" x="45.72" y="-22.86" rot="R180"/>
@@
 </segment>
 <segment>
-<pinref part="R23" gate="G$1" pin="2"/>
+<pinref part="1B" gate="G$1" pin="2"/>
 <pinref part="GND9" gate="1" pin="GND"/>
 <wire x1="142.24" y1="-167.64" x2="142.24" y2="-170.18" width="0.1524" layer="91"/>
@@
 <segment>
 <pinref part="GND7" gate="1" pin="GND"/>
-<pinref part="R19" gate="G$1" pin="2"/>
+<pinref part="5B" gate="G$1" pin="2"/>
 </segment>
 <segment>
@@
 <label x="160.02" y="-121.92" size="1.778" layer="95"/>
 <wire x1="160.02" y1="-121.92" x2="152.4" y2="-121.92" width="0.1524" layer="91"/>
-<pinref part="R20" gate="G$1" pin="2"/>
+<pinref part="J1" gate="G$1" pin="2"/>
 <wire x1="152.4" y1="-121.92" x2="152.4" y2="-109.22" width="0.1524" layer="91"/>
-<pinref part="R21" gate="G$1" pin="1"/>
+<pinref part="2A" gate="G$1" pin="1"/>
 <wire x1="142.24" y1="-129.54" x2="142.24" y2="-121.92" width="0.1524" layer="91"/>
 <junction x="142.24" y="-129.54"/>
-<pinref part="R14" gate="G$1" pin="1"/>
+<pinref part="4B" gate="G$1" pin="1"/>
 <wire x1="139.7" y1="-129.54" x2="142.24" y2="-129.54" width="0.1524" layer="91"/>
 <wire x1="152.4" y1="-121.92" x2="142.24" y2="-121.92" width="0.1524" layer="91"/>
@@
 <label x="142.24" y="-63.5" size="1.778" layer="95"/>
 <wire x1="142.24" y1="-68.58" x2="142.24" y2="-66.04" width="0.1524" layer="91"/>
-<pinref part="R11" gate="G$1" pin="1"/>
-<pinref part="R17" gate="G$1" pin="1"/>
+<pinref part="8B" gate="G$1" pin="1"/>
+<pinref part="4A" gate="G$1" pin="1"/>
 <wire x1="139.7" y1="-68.58" x2="142.24" y2="-68.58" width="0.1524" layer="91"/>
 <junction x="142.24" y="-68.58"/>
@@
 <segment>
 <pinref part="IC1" gate="D" pin="O"/>
-<pinref part="R14" gate="G$1" pin="2"/>
+<pinref part="4B" gate="G$1" pin="2"/>
 <wire x1="127" y1="-129.54" x2="129.54" y2="-129.54" width="0.1524" layer="91"/>
 </segment>
@@
 <segment>
 <pinref part="IC1" gate="E" pin="O"/>
-<pinref part="R15" gate="G$1" pin="2"/>
+<pinref part="3B" gate="G$1" pin="2"/>
 <wire x1="127" y1="-142.24" x2="129.54" y2="-142.24" width="0.1524" layer="91"/>
 </segment>
@@
 <segment>
 <pinref part="IC1" gate="F" pin="O"/>
-<pinref part="R16" gate="G$1" pin="2"/>
+<pinref part="2B" gate="G$1" pin="2"/>
 <wire x1="127" y1="-154.94" x2="129.54" y2="-154.94" width="0.1524" layer="91"/>
 </segment>
@@
 <net name="N$17" class="0">
 <segment>
-<pinref part="R23" gate="G$1" pin="1"/>
-<pinref part="R22" gate="G$1" pin="2"/>
+<pinref part="1B" gate="G$1" pin="1"/>
+<pinref part="1A" gate="G$1" pin="2"/>
 <wire x1="142.24" y1="-157.48" x2="142.24" y2="-154.94" width="0.1524" layer="91"/>
-<pinref part="R16" gate="G$1" pin="1"/>
+<pinref part="2B" gate="G$1" pin="1"/>
 <wire x1="142.24" y1="-154.94" x2="142.24" y2="-152.4" width="0.1524" layer="91"/>
 <wire x1="139.7" y1="-154.94" x2="142.24" y2="-154.94" width="0.1524" layer="91"/>
@@
 <net name="N$18" class="0">
 <segment>
-<pinref part="R15" gate="G$1" pin="1"/>
-<pinref part="R22" gate="G$1" pin="1"/>
+<pinref part="3B" gate="G$1" pin="1"/>
+<pinref part="1A" gate="G$1" pin="1"/>
 <wire x1="139.7" y1="-142.24" x2="142.24" y2="-142.24" width="0.1524" layer="91"/>
-<pinref part="R21" gate="G$1" pin="2"/>
+<pinref part="2A" gate="G$1" pin="2"/>
 <wire x1="142.24" y1="-142.24" x2="142.24" y2="-139.7" width="0.1524" layer="91"/>
 <junction x="142.24" y="-142.24"/>
@@
 <segment>
 <pinref part="IC1" gate="C" pin="O"/>
-<pinref part="R13" gate="G$1" pin="2"/>
+<pinref part="6B" gate="G$1" pin="2"/>
 <wire x1="127" y1="-93.98" x2="129.54" y2="-93.98" width="0.1524" layer="91"/>
 </segment>
@@
 <net name="N$21" class="0">
 <segment>
-<pinref part="R13" gate="G$1" pin="1"/>
+<pinref part="6B" gate="G$1" pin="1"/>
 <wire x1="139.7" y1="-93.98" x2="142.24" y2="-93.98" width="0.1524" layer="91"/>
-<pinref part="R18" gate="G$1" pin="2"/>
+<pinref part="3A" gate="G$1" pin="2"/>
 <wire x1="142.24" y1="-93.98" x2="142.24" y2="-91.44" width="0.1524" layer="91"/>
-<pinref part="R19" gate="G$1" pin="1"/>
+<pinref part="5B" gate="G$1" pin="1"/>
 <wire x1="142.24" y1="-93.98" x2="142.24" y2="-99.06" width="0.1524" layer="91"/>
 <junction x="142.24" y="-93.98"/>
-<pinref part="R20" gate="G$1" pin="1"/>
+<pinref part="J1" gate="G$1" pin="1"/>
 <wire x1="142.24" y1="-99.06" x2="152.4" y2="-99.06" width="0.1524" layer="91"/>
 <junction x="142.24" y="-99.06"/>
@@
 <segment>
 <pinref part="IC1" gate="B" pin="O"/>
-<pinref part="R12" gate="G$1" pin="2"/>
+<pinref part="7B" gate="G$1" pin="2"/>
 <wire x1="127" y1="-81.28" x2="129.54" y2="-81.28" width="0.1524" layer="91"/>
 </segment>
@@
 <net name="N$23" class="0">
 <segment>
-<pinref part="R12" gate="G$1" pin="1"/>
-<pinref part="R18" gate="G$1" pin="1"/>
+<pinref part="7B" gate="G$1" pin="1"/>
+<pinref part="3A" gate="G$1" pin="1"/>
 <wire x1="139.7" y1="-81.28" x2="142.24" y2="-81.28" width="0.1524" layer="91"/>
-<pinref part="R17" gate="G$1" pin="2"/>
+<pinref part="4A" gate="G$1" pin="2"/>
 <wire x1="142.24" y1="-81.28" x2="142.24" y2="-78.74" width="0.1524" layer="91"/>
 <junction x="142.24" y="-81.28"/>
@@
 <segment>
 <pinref part="IC1" gate="A" pin="O"/>
-<pinref part="R11" gate="G$1" pin="2"/>
+<pinref part="8B" gate="G$1" pin="2"/>
 <wire x1="127" y1="-68.58" x2="129.54" y2="-68.58" width="0.1524" layer="91"/>
 </segment>

Commit message: PCB V3
Parts:
- renumbered REG1 to IC2
Changed lines of the file:
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@@
 <part name="R9" library="rcl" deviceset="R-EU_" device="R0805"/>
 <part name="R10" library="rcl" deviceset="R-EU_" device="R0805"/>
-<part name="REG1" library="microbuilder" deviceset="VREG_SOT23" device=""/>
+<part name="IC2" library="microbuilder" deviceset="VREG_SOT23" device=""/>
 <part name="C2" library="rcl" deviceset="C-EU" device="C0805"/>
 <part name="GND8" library="supply1" deviceset="GND" device=""/>
@@
 <instance part="R9" gate="G$1" x="45.72" y="-22.86" rot="R180"/>
 <instance part="R10" gate="G$1" x="45.72" y="-25.4" rot="R180"/>
-<instance part="REG1" gate="G$1" x="162.56" y="-15.24"/>
+<instance part="IC2" gate="G$1" x="162.56" y="-15.24"/>
 <instance part="C2" gate="G$1" x="144.78" y="-22.86" smashed="yes">
 <attribute name="NAME" x="142.875" y="-19.558" size="1.778" layer="95" rot="R270"/>
@@
 </segment>
 <segment>
-<pinref part="REG1" gate="G$1" pin="GND"/>
+<pinref part="IC2" gate="G$1" pin="GND"/>
 <wire x1="152.4" y1="-17.78" x2="149.86" y2="-17.78" width="0.1524" layer="91"/>
 <wire x1="149.86" y1="-17.78" x2="149.86" y2="-35.56" width="0.1524" layer="91"/>
@@
 </segment>
 <segment>
-<pinref part="REG1" gate="G$1" pin="VOUT"/>
+<pinref part="IC2" gate="G$1" pin="VOUT"/>
 <wire x1="172.72" y1="-12.7" x2="182.88" y2="-12.7" width="0.1524" layer="91"/>
 <label x="180.34" y="-12.7" size="1.778" layer="95"/>
@@
 </segment>
 <segment>
-<pinref part="REG1" gate="G$1" pin="VIN"/>
+<pinref part="IC2" gate="G$1" pin="VIN"/>
 <wire x1="152.4" y1="-12.7" x2="144.78" y2="-12.7" width="0.1524" layer="91"/>
 <label x="134.62" y="-12.7" size="1.778" layer="95"/>
