File: oled_ui.sch (EAGLE design)
At the start: 42 parts, among them IC1 74HC14D

Commit message: pcb rev 4
Parts:
- removed 1A, 1B, 2A, 2B, 3A, 3B, 4A, 4B, 5B, 6B, 7B, 8B, J1, R3, R4, R5, R6, R7, R8: (no value), rcl:R-EU_R0805
- added C10: (no value), rcl:C-EUC0805
- added C8: 100n, rcl:C-EUC0805
- added ICSP: (no value), tag-connect:TC2030-MCP-NL
- added U$3, U$4, U$5, U$6, U$7, U$8: 0805DIODE, jasons_stuff:0805DIODE
- C1, C5, C6: value (none) -> 1u
- C3: value (none) -> 2u2
- C4: value (none) -> 4u7
- C7: value (none) -> 100n?
- IC1: value 74HC14D -> PIC12F1822SO08; device 74xx-eu:74HC14D -> jasons_stuff:PIC12F1822SO08
- IC2: value (none) -> MIC5504-2.8YM5-TR; device microbuilder:VREG_SOT23 -> jason_eagle6:MIC5504-2.8YM5-TR
- R1: value (none) -> 390k
- R10, R9: value (none) -> 4k7
- R2: value (none) -> 10k?
- renumbered C2 to C9
Connections:
- removed net BUTTONS_OUT1: 4A.1, 8B.1, JP2.3
- removed net BUTTONS_OUT2: 2A.1, 4B.1, J1.2, JP2.2
- removed net N$13: E.S, E.S1, IC1B.I, R4.1
- removed net N$15: 3B.2, IC1E.O
- removed net N$16: 2B.2, IC1F.O
- removed net N$17: 1A.2, 1B.1, 2B.1
- removed net N$18: 1A.1, 2A.2, 3B.1
- removed net N$20: 6B.2, IC1C.O
- removed net N$21: 3A.2, 5B.1, 6B.1, J1.1
- removed net N$22: 7B.2, IC1B.O
- removed net N$23: 3A.1, 4A.2, 7B.1
- removed net N$24: 8B.2, IC1A.O
- new net KEYA: IC1.RA5, U$3.P$2, U$4.P$2, U$5.P$2, U$6.P$1, U$7.P$1, U$8.P$1
- new net KEYB: D.P, D.P1, F.P, F.P1, IC1.RA4
- new net KEYC: C.P, C.P1, E.P, E.P1, IC1.MCLR#/VPP/RA3, ICSP.VPP/MCLR
- new net KEYD: A.P, A.P1, B.P, B.P1, IC1.RA0/PGD, ICSP.ICSP_DAT/PGD
- net 3V3: now also C10.1, C8.1, IC1.VDD, JP2.2
- net 5V: now also IC2.EN, ICSP.VDD; no longer IC1P.VCC, R3.2, R4.2, R5.2, R6.2, R7.2, R8.2
- net GND: now also C10.2, C8.2, IC1.VSS, ICSP.VSS(GND), JP2.3; no longer 1B.2, 5B.2, A.P, A.P1, B.P, B.P1, C.P, C.P1, D.P, D.P1, E.P, E.P1, F.P, F.P1, IC1P.GND
- net N$11: now also E.S, U$4.P$1; no longer C.S, C.S1, IC1D.I, R6.1
- net N$12: now also B.S, U$5.P$1; no longer D.S, D.S1, IC1C.I, R5.1
- net N$14: now also A.S, U$8.P$2; no longer F.S, F.S1, IC1A.I, R3.1
- net N$5: now also F.S, U$3.P$1; no longer B.S, B.S1, IC1F.I, R8.1
- net N$7: now also D.S, U$6.P$2; no longer 4B.2, IC1D.O
- net N$9: now also C.S, U$7.P$2; no longer A.S, A.S1, IC1E.I, R7.1
- net RST: now also JP1.3; no longer JP1.1
- net SCL: now also IC1.RA1/PGC, ICSP.ICSP_CLK/PGC
- net SDA: now also IC1.RA2, JP1.1; no longer JP1.3
Other:
- moved on the sheet: A, B, C, D, E, F
